Commit message: update

File: mobile_d/urdf/mobile_d.urdf (robot description, URDF)
Before this commit: robot mobile_d, 7 links, 6 joints
Joints:
- joint base_to_cam: origin xyz=0.2225 0 0.135 rpy=1.5708 0 0 -> xyz=0.2225 0 0.135 rpy=1.5708 0.7854 0
- joint base_to_lw: axis -1 0 0 -> 1 0 0
- joint base_to_rw: axis -1 0 0 -> 1 0 0

Commit message: model change

File: mobile_d/urdf/mobile_d.urdf (robot description, URDF)
Before this commit: robot mobile_d, 7 links, 6 joints
Joints:
- removed joint base_to_wheel_connector
- added joint base_to_connector: type fixed, parent base_link, child wheel_connector, origin xyz=0.073955 0 -0.013 rpy=1.5708 -6.123E-17 -1.5708, axis 0 0 0
- joint base_to_cam: origin xyz=0.2225 0 0.135 rpy=1.5708 0.7854 0 -> xyz=0.2225 0 0.135 rpy=1.5708 0 0
- joint base_to_lidar: axis 0 -1 0 -> 0 0 0; origin xyz=-0.025 -0.15 0.05 rpy=-1.5708 0 0 -> xyz=0.081395 -0.0065265 0.125 rpy=-1.5708 0 0

Commit message: model change_new

File: mobile_d/urdf/mobile_d.urdf (robot description, URDF)
Before this commit: robot mobile_d, 7 links, 6 joints
Links:
- link base_link: mass 40.5091303517493 -> 40.509
Joints:
- joint base_to_caster: origin xyz=-0.185 0 0 rpy=-1.5708 -3.5431E-18 -1.0846 -> xyz=-0.185 0 0 rpy=-1.5708 0 0
- joint base_to_connector: origin xyz=0.073955 0 -0.013 rpy=1.5708 -6.123E-17 -1.5708 -> xyz=0.076045 0 -0.013 rpy=1.5708 6.123E-17 1.5708
- joint base_to_lidar: axis 0 0 0 -> 0 1 0; origin xyz=0.081395 -0.0065265 0.125 rpy=-1.5708 0 0 -> xyz=-0.025 0.15 0.05 rpy=1.5708 0 0
- joint base_to_lw: axis 1 0 0 -> -1 0 0; origin xyz=0.073955 -0.148 -0.013 rpy=3.1416 6.123E-17 1.5708 -> xyz=0.076045 -0.148 -0.013 rpy=1.5708 6.123E-17 1.5708
- joint base_to_rw: axis 1 0 0 -> -1 0 0; origin xyz=0.073955 0.148 -0.013 rpy=3.1416 6.123E-17 1.5708 -> xyz=0.076045 0.148 -0.013 rpy=1.5708 6.123E-17 1.5708

Commit message: lidar_add

File: mobile_d/urdf/mobile_d.urdf (robot description, URDF)
Before this commit: robot mobile_d, 8 links, 7 joints
Links:
- added link vir_lidar
Joints:
- added joint vir_lidar_to_lidar: type fixed, parent lidar, child vir_lidar, origin xyz=0.10 0.04 0 rpy=1.5708 0 0, axis 0 0 0
- joint base_to_lw: axis 1 0 0 -> -1 0 0
- joint base_to_rw: axis 1 0 0 -> -1 0 0

Commit message: world_map

File: mobile_d/urdf/mobile_d.urdf (robot description, URDF)
Before this commit: robot mobile_d, 9 links, 8 joints
Joints:
- joint base_to_lw: axis -1 0 0 -> 1 0 0
- joint base_to_rw: axis -1 0 0 -> 1 0 0

Commit message: modle fin

File: mobile_d/urdf/mobile_d.urdf (robot description, URDF)
Before this commit: robot mobile_d, 9 links, 8 joints
Links:
- added link dumper, mass 15.275; collision mesh filename=package://mobile_d/meshes/dumper.STL; visual mesh filename=package://mobile_d/meshes/dumper.STL
- link base_link: mass 40.613 -> 41.2800177633281
Joints:
- added joint base_to_dumper: type revolute, parent base_link, child dumper, origin xyz=-0.18 0 0.0855 rpy=1.5708 0 3.1416, axis 0 0 -1, limit lower=0 upper=1.2217 effort=0 velocity=0
- joint base_to_cam: axis 0 1 0 -> 0 0 1

Commit message: dump

File: mobile_d/urdf/mobile_d.urdf (robot description, URDF)
Before this commit: robot mobile_d, 10 links, 9 joints
Joints:
- joint base_to_dumper: limit lower=0 upper=1.2217 effort=0 velocity=0 -> lower=0 upper=1.2217 effort=300 velocity=1

Commit message: model update

File: mobile_d/urdf/mobile_d.urdf (robot description, URDF)
Before this commit: robot mobile_d, 10 links, 9 joints
Links:
- link dumper: mass 15.275 -> 0.015275
